Commit message: edits to iiwa safety control

File: urdf/iiwa7.xacro (robot description, xacro)
@@ -53,8 +53,8 @@
       <origin xyz="0 0 0.15" rpy="0 0 0"/>
       <axis xyz="0 0 1"/>
-      <limit lower="${-170 * PI / 180}" upper="${170 * PI / 180}"
-             effort="${max_effort}" velocity="${max_velocity}" />
-      <safety_controller soft_lower_limit="${-168 * PI / 180}"
-                         soft_upper_limit="${168 * PI / 180}"
+      <limit lower="${-165 * PI / 180}" upper="${165 * PI / 180}"
+             effort="${max_effort}" velocity="${max_velocity}" />
+      <safety_controller soft_lower_limit="${-165 * PI / 180}"
+                         soft_upper_limit="${165 * PI / 180}"
                          k_position="${safety_controller_k_pos}"
                          k_velocity="${safety_controller_k_vel}"/>
@@ -87,8 +87,8 @@
       <origin xyz="0 0 0.19" rpy="${PI / 2}   0 ${PI}"/>
       <axis xyz="0 0 1"/>
-      <limit lower="${-120 * PI / 180}" upper="${120 * PI / 180}"
-             effort="${max_effort}" velocity="${max_velocity}" />
-      <safety_controller soft_lower_limit="${-118 * PI / 180}"
-                         soft_upper_limit="${118 * PI / 180}"
+      <limit lower="${-115 * PI / 180}" upper="${115 * PI / 180}"
+             effort="${max_effort}" velocity="${max_velocity}" />
+      <safety_controller soft_lower_limit="${-115 * PI / 180}"
+                         soft_upper_limit="${115 * PI / 180}"
                          k_position="${safety_controller_k_pos}"
                          k_velocity="${safety_controller_k_vel}"/>
@@ -121,8 +121,8 @@
       <origin xyz="0 0.21 0" rpy="${PI / 2} 0 ${PI}"/>
       <axis xyz="0 0 1"/>
-      <limit lower="${-170 * PI / 180}" upper="${170 * PI / 180}"
-             effort="${max_effort}" velocity="${max_velocity}" />
-      <safety_controller soft_lower_limit="${-168 * PI / 180}"
-                         soft_upper_limit="${168 * PI / 180}"
+      <limit lower="${-165 * PI / 180}" upper="${165 * PI / 180}"
+             effort="${max_effort}" velocity="${max_velocity}" />
+      <safety_controller soft_lower_limit="${-165 * PI / 180}"
+                         soft_upper_limit="${165 * PI / 180}"
                          k_position="${safety_controller_k_pos}"
                          k_velocity="${safety_controller_k_vel}"/>
@@ -155,8 +155,8 @@
       <origin xyz="0 0 0.19" rpy="${PI / 2} 0 0"/>
       <axis xyz="0 0 1"/>
-      <limit lower="${-120 * PI / 180}" upper="${120 * PI / 180}"
-             effort="${max_effort}" velocity="${max_velocity}" />
-      <safety_controller soft_lower_limit="${-118 * PI / 180}"
-                         soft_upper_limit="${118 * PI / 180}"
+      <limit lower="${-115 * PI / 180}" upper="${115 * PI / 180}"
+             effort="${max_effort}" velocity="${max_velocity}" />
+      <safety_controller soft_lower_limit="${-115 * PI / 180}"
+                         soft_upper_limit="${115 * PI / 180}"
                          k_position="${safety_controller_k_pos}"
                          k_velocity="${safety_controller_k_vel}"/>
@@ -189,8 +189,8 @@
       <origin xyz="0 0.21 0" rpy="${-PI / 2} ${PI} 0"/>
       <axis xyz="0 0 1"/>
-      <limit lower="${-170 * PI / 180}" upper="${170 * PI / 180}"
-             effort="${max_effort}" velocity="${max_velocity}" />
-      <safety_controller soft_lower_limit="${-168 * PI / 180}"
-                         soft_upper_limit="${168 * PI / 180}"
+      <limit lower="${-165 * PI / 180}" upper="${165 * PI / 180}"
+             effort="${max_effort}" velocity="${max_velocity}" />
+      <safety_controller soft_lower_limit="${-165 * PI / 180}"
+                         soft_upper_limit="${165 * PI / 180}"
                          k_position="${safety_controller_k_pos}"
                          k_velocity="${safety_controller_k_vel}"/>
@@ -223,8 +223,8 @@
       <origin xyz="0 0.06070 0.19" rpy="${PI / 2} 0 0"/>
       <axis xyz="0 0 1"/>
-      <limit lower="${-120 * PI / 180}" upper="${120 * PI / 180}"
-             effort="${max_effort}" velocity="${max_velocity}" />
-      <safety_controller soft_lower_limit="${-118 * PI / 180}"
-                         soft_upper_limit="${118 * PI / 180}"
+      <limit lower="${-115 * PI / 180}" upper="${115 * PI / 180}"
+             effort="${max_effort}" velocity="${max_velocity}" />
+      <safety_controller soft_lower_limit="${-115 * PI / 180}"
+                         soft_upper_limit="${115 * PI / 180}"
                          k_position="${safety_controller_k_pos}"
                          k_velocity="${safety_controller_k_vel}"/>
@@ -257,8 +257,8 @@
       <origin xyz="0 0.081 0.06070" rpy="${- PI / 2} ${PI} 0"/>
       <axis xyz="0 0 1"/>
-      <limit lower="${-175 * PI / 180}" upper="${175 * PI / 180}"
-             effort="${max_effort}" velocity="${max_velocity}" />
-      <safety_controller soft_lower_limit="${-173 * PI / 180}"
-                         soft_upper_limit="${173 * PI / 180}"
+      <limit lower="${-170 * PI / 180}" upper="${170 * PI / 180}"
+             effort="${max_effort}" velocity="${max_velocity}" />
+      <safety_controller soft_lower_limit="${-170 * PI / 180}"
+                         soft_upper_limit="${170 * PI / 180}"
                          k_position="${safety_controller_k_pos}"
                          k_velocity="${safety_controller_k_vel}"/>
